Commit message: 2square_motion.py

File: urdf/_d435.urdf.xacro (robot description, xacro)
@@ -56,5 +56,7 @@
         <origin xyz="0 ${-d435_cam_depth_py} 0" rpy="0 0 0"/>
         <geometry>
-        <box size="${d435_cam_depth} ${d435_cam_width} ${d435_cam_height}"/>
+        <!-- <box size="${d435_cam_depth} ${d435_cam_width} ${d435_cam_height}"/> -->
+        <box size="0.05 0.05 0.05"/>
+        <!-- <box size="0.001 0.001 0.001"/> -->
         </geometry>
       </collision>
